Commit message: robot moving

File: description/robot_core.xacro (robot description, xacro)
@@ -41,4 +41,7 @@
         </xacro:inertial_box>
     </link>
+    <gazebo reference="chassis">
+        <material>Gazebo/White</material>
+    </gazebo>
     <!-- LEFT WHEEL LINK -->
     <joint name="left_wheel_joint" type="continuous">
@@ -64,4 +67,7 @@
         </xacro:inertial_cylinder>
     </link>
+     <gazebo reference="left_wheel">
+        <material>Gazebo/Blue</material>
+    </gazebo>
     <!-- RIGHT WHEEL LINK -->
     <joint name="right_wheel_joint" type="continuous">
@@ -87,4 +93,7 @@
         </xacro:inertial_cylinder>
     </link>
+    <gazebo reference="right_wheel">
+        <material>Gazebo/Blue</material>
+    </gazebo>
     <!-- CASTER WHEEL LINK -->
     <joint name="caster_wheel_joint" type="fixed">
@@ -109,3 +118,8 @@
         </xacro:inertial_sphere>
     </link>
+    <gazebo reference="caster_wheel">
+        <material>Gazebo/Black</material>
+        <mu1 value="0.001"/>
+        <mu2 value="0.001"/>
+    </gazebo>
 </robot>

Commit message: name tag

File: description/robot_core.xacro (robot description, xacro)
@@ -44,4 +44,16 @@
         <material>Gazebo/White</material>
     </gazebo>
+    <link name="name_tag">
+        <visual>
+            <geometry>
+                <mesh filename="package://my_bot/meshes/BHAVYA.stl" scale="0.002 0.002 0.002" />
+            </geometry>
+        </visual>
+    </link>
+    <joint name="name_tag_joint" type="fixed">
+        <parent link="base_link"/>
+        <child link="name_tag"/>
+        <origin xyz="0 0 0.190"/>
+    </joint>
     <!-- LEFT WHEEL LINK -->
     <joint name="left_wheel_joint" type="continuous">

Commit message: name file

File: description/robot_core.xacro (robot description, xacro)
@@ -54,5 +54,5 @@
         <parent link="base_link"/>
         <child link="name_tag"/>
-        <origin xyz="0 0 0.190"/>
+        <origin xyz="0 0 0.157"/>
     </joint>
     <!-- LEFT WHEEL LINK -->
